File: PCB/All-in-one/All-in-one.kicad_sch (KiCad schematic)
At the start: 4 parts, among them U1 MPU6050, U2 BMP280, U3 NEO-6M-GPS, U4 STM32F401CCUx

Commit message: Update
Parts:
- added C? (x2): 0.1u F, symbol pspice:CAP
- added C?: 2n2, symbol pspice:CAP
Connections:
- net at U1.10 (REGOUT): now also C?.1
- net VDD: now reaches U1.13 (VDD)
- net VDD: now also C?.1
- net GND: now reaches U1.18 (GND)
- net GND: now also C?.2, C?.2, C?.2
- net at U1.20 (CPOUT): now also C?.1
Other:
- note added: "MPU6050 Pinout"
- moved on the sheet: U1

Commit message: Added draft schematic and STM32CubeIDE Project - Added all datasheets
- Started schematic draftin

- Started STM32C
Parts:
- removed U4: STM32F401CCUx, Package_DFN_QFN:QFN-48-1EP_7x7mm_P0.5mm_EP5.6x5.6mm, symbol MCU_ST_STM32F4:STM32F401CCUx
- added C?: 2u2, symbol Device:C_Small
- added C?: 10n, symbol Device:C_Small
- added C?: 4u7, symbol Device:C_Small
- added C? (x4): 100n, symbol Device:C_Small
- added C? (x2): 12p, symbol Device:C_Small
- added C?: 1u, symbol Device:C_Small
- added C?: u1, symbol Device:C_Small
- added D?: LED_BLUE, symbol Device:LED
- added L?: 39n, symbol Device:L_Small
- added R?: 1k5, symbol Device:R_Small
- added R?: 0, symbol Device:R_Small
- added R?: 10k, symbol Device:R_Small
- added SW? (x2): SW_Push, symbol Switch:SW_Push
- added U?: STM32F401CDUx, Package_DFN_QFN:QFN-48-1EP_7x7mm_P0.5mm_EP5.6x5.6mm, symbol MCU_ST_STM32F4:STM32F401CDUx
- added Y?: 25MHz 12pF, symbol Device:Crystal_GND24_Small
Connections:
- net GND: now also C?.1, C?.2, C?.2, C?.2, C?.2, C?.2, C?.2, C?.2, C?.2, C?.2, C?.2, R?.2, SW?.1, SW?.2, U?.23 (VSS), U?.35 (VSS), U?.44 (BOOT0), U?.47 (VSS), U?.49 (VSS), U?.8 (VSSA), Y?.2, Y?.4
- new net: C?.1, U?.22 (VCAP1)
- new net: D?.1 (K), R?.1
- new net: R?.2, SW?.1
- new net: C?.1, R?.2, Y?.3
- new net +3.3V: C?.1, C?.1, C?.1, C?.1, C?.1, L?.1, R?.1, U?.1 (VBAT), U?.24 (VDD), U?.36 (VDD), U?.48 (VDD)
- new net +3.3VA: C?.1, C?.1, L?.2, U?.9 (VREF+/VDDA)
- new net HSE_IN: C?.1, U?.5 (PH0), Y?.1
- new net HSE_OUT: R?.1, U?.6 (PH1)
- new net I2C1_SCL: U?.16 (PA6)
- new net I2C1_SDA: U?.17 (PA7)
- new net LED_STATUS: D?.2 (A), U?.20 (PB2)
- new net NRST: C?.2, SW?.2, U?.7 (NRST)
- new net SWCLK: U?.37 (PA14)
- new net SWDIO: U?.34 (PA13)
- new net SWO: U?.39 (PB3)
- new net UART2_RX: U?.13 (PA3)
- new net UART2_TX: U?.12 (PA2)
- new net USB_D+: U?.33 (PA12)
- new net USB_D-: U?.32 (PA11)
- no-connect marks 0 -> 24
Other:
- note added: "CHECK EXTERNAL RESISTOR VALUE"
- note added: "CHECK PWM PINS FOR SERVO /EXTERNAL MOTOR CONNECTION"
- note added: "C_LOAD = 2*(C_L - C_STARY) = 2*(12pF - (5-6pF)) = 12pF C_LOAD is single load cap value C_L is given by manufractuer C_STRAY is the capacitacne of the board (5-6 pF by research)"
- note added: "Decoupling Caps A single 4u7 and 100n per VBAT/VDD Each 100n Cap should place as close as the chip as possible in PCB layout"
- note added: "Low Pass Filter on VDDA, extra filtering on V_Analog"
- note added: "NRST pin protection as suggested (Note that NRST has a internal weak pullup to ensure it is always HIGH (TRUE) to prevent unwanted reset)"
- note added: "Pin pull down, BOOT0 HIGH = Program mode"
- note added: "X322525MOB4SI"
- note removed: "Add decoupling"
- company: (none) -> GORDON SO
- title: (none) -> ALL-IN-ONE
- moved on the sheet: U2, U3

Commit message: Draft Schematic - Schematic is 80%ish done, details on minor connections need more research - Wired sensors - Added extra connectors - SD card slot is NOT wired
Parts:
- removed C? (x2): 0.1u F, symbol pspice:CAP
- removed C?: 2n2, symbol pspice:CAP
- removed U1: MPU6050, IC_MPU6050, symbol MPU:MPU6050
- removed U2: BMP280, XDCR_BMP280, symbol BMP:BMP280
- added C? (x5): u1, symbol Device:C_Small
- added C? (x2): 10u, symbol Device:C_Small
- added C? (x2): 22u, symbol Device:C_Small
- added C?: 10n, symbol Device:C_Small
- added C?: 2n2, symbol Device:C_Small
- added D?: B5819W, symbol Device:D_Schottky_Small
- added F?: 250mA, symbol Device:Polyfuse
- added FB?: 600 @ 600MHz, symbol Device:FerriteBead_Small
- added H? (x4): MountingHole, symbol Mechanical:MountingHole
- added J?: LOW VOLTAGE, symbol Connector:Screw_Terminal_01x02
- added J?: USB_C_Receptacle_USB2.0, symbol Connector:USB_C_Receptacle_USB2.0
- added J?: HIGH VOLTAGE, symbol Connector:Screw_Terminal_01x02
- added J?: SWD, symbol Connector_Generic:Conn_02x05_Odd_Even
- added J?: I2C_EXT, symbol Connector_Generic:Conn_01x04
- added J?: UART_EXT, symbol Connector_Generic:Conn_01x04
- added J?: Micro_SD_Card, symbol Connector:Micro_SD_Card
- added L?: 2u2, symbol Device:L_Small
- added Q?: AO3401A, Package_TO_SOT_SMD:SOT-23, symbol Transistor_FET:AO3401A
- added R?: 33k, symbol Device:R_Small
- added R? (x2): 5k1, symbol Device:R_Small
- added R?: 10k, symbol Device:R_Small
- added R? (x2): 2k2, symbol Device:R_Small
- added R?: 200, symbol Device:R_Small
- added U?: USBLC6-2P6, Package_TO_SOT_SMD:SOT-666, symbol Power_Protection:USBLC6-2P6
- added U?: BMP280, Package_LGA:Bosch_LGA-8_2x2.5mm_P0.65mm_ClockwisePinNumbering, symbol Sensor_Pressure:BMP280
- added U?: MPU-6050, Sensor_Motion:InvenSense_QFN-24_4x4mm_P0.5mm, symbol Sensor_Motion:MPU-6050
- added U?: TPS563201DDCR, Package_TO_SOT_SMD:SOT-23-6, symbol Regulator_Switching:TPS563200
Connections:
- net +3.3V: now also C?.1, C?.1, C?.1, C?.1, C?.2, C?.2, J?.1 (Pin_1), J?.1 (Pin_1), J?.1 (Pin_1), L?.2, R?.1, R?.2, R?.2, U?.13 (VDD), U?.2 (CSB), U?.6 (VDDIO), U?.8 (VDD), U?.8 (VDDIO)
- net GND: now also C?.1, C?.1, C?.2, C?.2, C?.2, C?.2, C?.2, C?.2, C?.2, C?.2, J?.2 (Pin_2), J?.3 (Pin_3), J?.4 (Pin_4), J?.4 (Pin_4), J?.5 (Pin_5), J?.9 (Pin_9), J?.A1 (GND), J?.A12 (GND), J?.B1 (GND), J?.B12 (GND), Q?.1 (G), R?.2, R?.2, R?.2, U?.1 (GND), U?.1 (GND), U?.18 (GND), U?.2 (GND), U?.5 (SDO), U?.7 (GND)
- net I2C1_SCL: now also J?.2 (Pin_2), R?.1, U?.24 (SDA), U?.4 (SCK)
- net I2C1_SDA: now also J?.3 (Pin_3), R?.1, U?.23 (SCL), U?.3 (SDI)
- net NRST: now also J?.10 (Pin_10)
- net SWCLK: now also J?.4 (Pin_4)
- net SWDIO: now also J?.2 (Pin_2)
- net SWO: now also J?.6 (Pin_6)
- net UART2_RX: now also J?.3 (Pin_3)
- net UART2_TX: now also J?.2 (Pin_2)
- net USB_D+: now also U?.4 (I/O2)
- net USB_D-: now also U?.6 (I/O1)
- new net: R?.1, R?.2
- new net: D?.1 (K), FB?.1, Q?.2 (S)
- new net: C?.1, C?.1, FB?.2, U?.3 (VIN), U?.5 (EN)
- new net: F?.2, Q?.3 (D)
- new net: C?.1, U?.10 (REGOUT)
- new net: C?.1, U?.20 (CPOUT)
- new net +12V: F?.1, J?.1 (Pin_1)
- new net +5V: D?.2 (A), J?.A4 (VBUS), J?.A9 (VBUS), J?.B4 (VBUS), J?.B9 (VBUS), U?.5 (VBUS)
- new net BUCK_SW: C?.1, L?.1, U?.2 (SW)
- new net BUCK_VBST: C?.2, U?.6 (VBST)
- new net BUCK_VFB: R?.1, R?.2, U?.4 (VFB)
- new net USBC_CONNCC1: J?.A5 (CC1), R?.1
- new net USBC_CONNCC2: J?.B5 (CC2), R?.1
- new net USBC_CONND+: J?.A6 (D+), J?.B6 (D+), U?.3 (I/O2)
- new net USBC_CONND-: J?.A7 (D-), J?.B7 (D-), U?.1 (I/O1)
- no-connect marks 24 -> 29
Other:
- note added: "3 POWER INPUT 1* Normal (Lipo ~3.3-5V input) 2* High V (4.5V-12V input/USB 5V)"
- note added: "Blue LED foward voltage ~3V"
- note added: "Buck Converter"
- note added: "ESP to protect the board"
- note added: "Extra connectors for possible needs"
- note added: "I2C Address bit 0 = '0'"
- note added: "I2C Pull Up (PU) Resistors Value is by research, verified with I2C Application Report by Texas Instruments (SLVA689) R_P(MAX) = t_rise_max/(0.8473*C_bus) t_rise_max = 1000ns (I2C Standard Mode)/C_bus = 400pF (by datasheet) R_P(MAX) = 1000ns/(0.8473*400pF) = 2951 ohm *The R_P(max) is related to the capacitve nature of the bus line, the higher the Pull-up resistor, the higher of the time constant (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"
- note added: "PD Resistor for Upstream Facing Port (UFP) This port is to decide the orientation of the USBC cable"
- note added: "STM32 MCU"
- note added: "This connecter is for debug and flash the code through a universal 10pin Cortex Debuger Users can use a ST-LINK with the correct pin connection"
- note added: "Values are choosen from datasheet and research"
- moved on the sheet: D?, R?

Commit message: Minor Update
Parts:
- removed J?: Micro_SD_Card, symbol Connector:Micro_SD_Card
- added J?: Micro_SD_Card_Det, symbol Connector:Micro_SD_Card_Det
Changed lines of the file:
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@@
     (pin "1")
+  )
+  (symbol (lib_id "Connector:Micro_SD_Card_Det") (at 133.35 163.83 0) (unit 1)
+    (in_bom yes) (on_board yes) (fields_autoplaced)
+    (property "Reference" "J?" (id 0) (at 133.985 142.24 0))
+    (property "Value" "Micro_SD_Card_Det" (id 1) (at 133.985 144.78 0))
+    (property "Footprint" "" (id 2) (at 185.42 146.05 0)
+      (effects (font (size 1.27 1.27)) hide)
+    )
+    (property "Datasheet" "https://www.hirose.com/product/en/download_file/key_name/DM3/category/Catalog/doc_file_id/49662/?file_category_id=4&item_id=195&is_series=1" (id 3) (at 133.35 161.29 0)
+      (effects (font (size 1.27 1.27)) hide)
+    )
+    (pin "1")
+    (pin "10")
+    (pin "11")
+    (pin "2")
+    (pin "3")
+    (pin "4")
+    (pin "5")
+    (pin "6")
+    (pin "7")
+    (pin "8")
+    (pin "9")
   )
   (symbol (lib_id "Device:C_Small") (at 158.75 114.3 0) (unit 1)
@@
     (pin "1")
   )
-  (symbol (lib_id "Connector:Micro_SD_Card") (at 154.94 158.75 0) (unit 1)
-    (in_bom yes) (on_board yes) (fields_autoplaced)
-    (property "Reference" "J?" (id 0) (at 155.575 140.97 0))
-    (property "Value" "Micro_SD_Card" (id 1) (at 155.575 143.51 0))
-    (property "Footprint" "" (id 2) (at 184.15 151.13 0)
-      (effects (font (size 1.27 1.27)) hide)
-    )
-    (property "Datasheet" "http://katalog.we-online.de/em/datasheet/693072010801.pdf" (id 3) (at 154.94 158.75 0)
-      (effects (font (size 1.27 1.27)) hide)
-    )
-    (pin "1")
-    (pin "2")
-    (pin "3")
-    (pin "4")
-    (pin "5")
-    (pin "6")
-    (pin "7")
-    (pin "8")
-    (pin "9")
-  )
   (symbol (lib_id "Device:LED") (at 306.07 172.72 180) (unit 1)
     (in_bom yes) (on_board yes) (fields_autoplaced)
@@
       (reference "J?") (unit 1) (value "SWD") (footprint "")
     )
+    (path "/c8638e45-d05e-45c0-8ab5-690e9bbe595a"
+      (reference "J?") (unit 1) (value "Micro_SD_Card_Det") (footprint "")
+    )
     (path "/d69f8787-4d65-4c5b-ac9f-6cf47c3c3de8"
       (reference "J?") (unit 1) (value "I2C_EXT") (footprint "")
@@
       (reference "J?") (unit 1) (value "UART_EXT") (footprint "")
     )
-    (path "/f2a10124-8992-4a33-8d4f-44747dcf4ceb"
-      (reference "J?") (unit 1) (value "Micro_SD_Card") (footprint "")
-    )
     (path "/4886908c-bfd1-45f0-89b1-f1d97145c505"

Commit message: Pin Finalize and Added SD Card Slot Via SPI - Pin and circuit are ready to final check - Added LDO for Lipo, a power source switch should be added
Parts:
- removed U3: NEO-6M-GPS, XCVR_NEO-6M-GPS, symbol NEO6M:NEO-6M-GPS
- added C? (x2): 22u, symbol Device:C_Small
- added J?: TIM, symbol Connector_Generic:Conn_01x04
- added J?: GPIO, symbol Connector_Generic:Conn_01x04
- added R? (x2): 10k, symbol Device:R_Small
- added U?: AMS1117-3.3, Package_TO_SOT_SMD:SOT-223-3_TabPin2, symbol Regulator_Linear:AMS1117-3.3
- C?: value 2u2 -> 4u7
Connections:
- net +3.3V: now also J?.4 (VDD), C?.2, R?.2, R?.2, U?.2 (VO)
- net GND: now also J?.11 (SHIELD), J?.2 (Pin_2), J?.6 (VSS), C?.1, C?.1, J?.3 (Pin_3), J?.4 (Pin_4), U?.1 (GND)
- net I2C1_SCL: now also U?.42 (PB6); no longer U?.16 (PA6)
- net I2C1_SDA: now also U?.43 (PB7); no longer U?.17 (PA7)
- net UART2_RX: now also U?.31 (PA10); no longer U?.13 (PA3)
- net UART2_TX: now also U?.30 (PA9); no longer U?.12 (PA2)
- net +BATT: now reaches J?.1 (Pin_1)
- net +BATT: now also C?.2, U?.3 (VI)
- net TIM2_CH1: now reaches U?.10 (PA0)
- net TIM2_CH1: now also J?.1 (Pin_1)
- net SPI1_NSS: now reaches U?.14 (PA4)
- net SPI1_NSS: now also J?.2 (DAT3/CD)
- net SPI1_SCK: now reaches U?.15 (PA5)
- net SPI1_SCK: now also J?.5 (CLK)
- net SD_CARD_DET: now reaches U?.18 (PB0)
- net SD_CARD_DET: now also J?.9 (DET_B), R?.1
- net GPIO_1: now reaches U?.25 (PB12)
- net GPIO_1: now also J?.1 (Pin_1)
- net GPIO_2: now reaches U?.26 (PB13)
- net GPIO_2: now also J?.2 (Pin_2)
- net GPIO_3: now reaches U?.27 (PB14)
- net GPIO_3: now also J?.3 (Pin_3)
- net GPIO_4: now reaches U?.28 (PB15)
- net GPIO_4: now also J?.4 (Pin_4)
- net MPU_INT: now reaches U?.41 (PB5)
- net MPU_INT: now also U?.12 (INT)
- net SPI1_MOSI: now reaches J?.3 (CMD)
- net SPI1_MOSI: now also U?.17 (PA7)
- net SPI1_MISO: now reaches J?.7 (DAT0)
- net SPI1_MISO: now also U?.16 (PA6), R?.1
- new net TIM5_CH1: J?.2 (Pin_2), U?.12 (PA2)
- no-connect marks 29 -> 24
Other:
- note added: "SPI MISO pullup Only MISO is a input pin on the MCU side, PU resistor is a must in SPI as it is not a drain type like I2C"
- note added: "TIMer can be configured anyway for general purpose TIM pins are chosen to keep PWM output"
- note removed: "CHECK PWM PINS FOR SERVO /EXTERNAL MOTOR CONNECTION"
- note removed: "MPU6050 Pinout"
- moved on the sheet: C?, J?, U?

Commit message: REV X01 Schematic Completed - Schematic is completed, with the purpose of X01 being the proto board - External resistor of the external clock is left as a pad only, it is a bit unclear that if a external resistor is a must, when ordering the PCB this is not a issue as we can just buy extra SMD resistor - All labels applied and passed ERC - Added LDO for Lipo
Parts:
- removed C? (x2): 22u, symbol Device:C_Small
- removed U?: AMS1117-3.3, Package_TO_SOT_SMD:SOT-223-3_TabPin2, symbol Regulator_Linear:AMS1117-3.3
- added C6: 10u, symbol Device:C_Small
- added C7, C8: u1, symbol Device:C_Small
- added D2: LED_RED, symbol Device:LED
- added D3: LED_BLUE, symbol Device:LED
- added R4: 1k5, symbol Device:R_Small
- added SW1: SW_DPDT_x2, symbol Switch:SW_DPDT_x2
- added U2: NCP114AMX330TCG, symbol All-in-one_custom:NCP114AMX330TCG
- D4: renamed from D?; value LED_BLUE -> LED_GREEN
- gave numbers to parts that had none: 60
Connections:
- net +3.3V: now also SW1.2 (B); no longer C4.2, C5.2, L1.2
- net +BATT: now also C6.1, C7.1, U2.3 (EN), U2.4 (IN)
- net GND: now also C6.2, C7.2, C8.2, R4.2, U2.2 (GND)
- new net: D2.1 (K), SW1.4 (A)
- new net: R4.1, SW1.5 (B)
- new net: D3.1 (K), SW1.6 (C)
- new net +3.3V (HIGH V): C4.2, C5.2, D2.2 (A), L1.2, SW1.1 (A)
- new net +3.3V (LOW V): C8.1, D3.2 (A), SW1.3 (C), U2.1 (OUT)
- no-connect marks 24 -> 26
Other:
- note added: "CONNECTORS"
- note added: "DEBUG/FLASH"
- note added: "EXTRA CONNECTORS"
- note added: "I2C"
- note added: "LDO"
- note added: "POWER"
- note added: "SPI"
- note added: "USB"
- note removed: "Extra connectors for possible needs"
- moved on the sheet: C20, C21, C22, C23, C24, C25, C4, C5, D1, H1, H2, J2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

Commit message: Updated Schematic and Footprint Assignments
- Updated power supply circuit switch
- Added custom foot prints
- Assigned most of the footprints
Parts:
- removed D3: LED_BLUE, symbol Device:LED
- removed H1, H2, H3, H4: MountingHole, symbol Mechanical:MountingHole
- removed J6: TIM, symbol Connector_Generic:Conn_01x04
- removed SW1: SW_DPDT_x2, symbol Switch:SW_DPDT_x2
- added H1, H2, H3, H4: MountingHole_Pad, MountingHole:MountingHole_3.5mm_Pad_Via, symbol Mechanical:MountingHole_Pad
- added J6, J7: Conn_01x02, Connector_PinHeader_2.54mm:PinHeader_1x02_P2.54mm_Vertical, symbol Connector_Generic:Conn_01x02
- added SW1: SW_DP3T, All-in-one-custom:SMNR4020-2.2UH, symbol Switch:SW_DP3T
- C1, C4, C5, C6: footprint (none) -> Capacitor_SMD:C_1206_3216Metric
- C10, C13, C14, C15, C16, C17, C18, C22, C25: footprint (none) -> Capacitor_SMD:C_0402_1005Metric
- C11, C12, C19, C20: footprint (none) -> Capacitor_SMD:C_0603_1608Metric
- C2, C3, C7, C8: value u1 -> 100n; footprint (none) -> Capacitor_SMD:C_0805_2012Metric
- C21, C23, C24, C9: value u1 -> 100n; footprint (none) -> Capacitor_SMD:C_0402_1005Metric
- D1: footprint (none) -> Diode_SMD:D_SOD-123
- D2, D4: footprint (none) -> LED_SMD:LED_0402_1005Metric
- F1: footprint (none) -> Fuse:Fuse_1206_3216Metric
- FB1: footprint (none) -> Inductor_SMD:L_1206_3216Metric
- J1, J2: footprint (none) -> TerminalBlock_TE-Connectivity:TerminalBlock_TE_282834-2_1x02_P2.54mm_Horizontal
- J10: renamed from J9; footprint (none) -> Connector_PinHeader_2.54mm:PinHeader_2x05_P2.54mm_Vertical
- J5: footprint (none) -> Connector_PinHeader_2.54mm:PinHeader_1x04_P2.54mm_Vertical
- J8: renamed from J7; footprint (none) -> Connector_PinHeader_2.54mm:PinHeader_1x04_P2.54mm_Vertical
- J9: renamed from J8; footprint (none) -> Connector_PinHeader_2.54mm:PinHeader_1x04_P2.54mm_Vertical
- L1: footprint (none) -> All-in-one-custom:SMNR4020-2.2UH; PART ID (none) -> SMNR4020-2.2UH
- L2: footprint (none) -> Inductor_SMD:L_0402_1005Metric
- R1, R2, R3, R4: footprint (none) -> Resistor_SMD:R_0603_1608Metric
- R10: renamed from R9; footprint (none) -> Resistor_SMD:R_0603_1608Metric
- R11: renamed from R10; footprint (none) -> Resistor_SMD:R_0402_1005Metric
- R12: renamed from R11; footprint (none) -> Resistor_SMD:R_0402_1005Metric
- R13: renamed from R12; footprint (none) -> Resistor_SMD:R_0402_1005Metric
- R5: footprint (none) -> Resistor_SMD:R_0402_1005Metric
- R6: renamed from R?; value 0 -> 510; footprint (none) -> Resistor_SMD:R_0402_1005Metric
- R7: renamed from R6; footprint (none) -> Resistor_SMD:R_0603_1608Metric
- R8: renamed from R7; footprint (none) -> Resistor_SMD:R_0402_1005Metric
- R9: renamed from R8; footprint (none) -> Resistor_SMD:R_0603_1608Metric
- U2: footprint (none) -> Package_DFN_QFN:UDFN-4-1EP_1x1mm_P0.65mm_EP0.48x0.48mm
- Y1: footprint (none) -> Crystal:Crystal_SMD_3225-4Pin_3.2x2.5mm; PART ID (none) -> X322525MOB4SI
Connections:
- net +3.3V (HIGH V) is gone; now on net +3.3V: C4.2, C5.2, D2.2 (A), L1.2
- net +3.3V (LOW V) is gone; now on net +3.3V: C8.1, U2.1 (OUT)
- net +BATT: now also SW1.7, SW1.8
- net GND: now also H1.1, H2.1, H3.1, H4.1, J6.2 (Pin_2), J7.2 (Pin_2)
- net TIM2_CH1: now also J6.1 (Pin_1)
- net TIM5_CH1: now also J7.1 (Pin_1)
- net at D2.1 (K): now also R4.1
- net BUCK_VIN: now reaches C1.1, C2.1, FB1.2, U1.3 (VIN), U1.5 (EN)
- net BUCK_VIN: now also SW1.1, SW1.3
- no-connect marks 26 -> 29
Other:
- note added: "C_LOAD = 2*(C_L - C_STARY) = 2*(12pF - (5-6pF)) = 12pF C_LOAD is single load cap value C_L is given by manufractuer C_STRAY is the capacitacne of the board (5-6 pF by research) R6 is the external resistor in the circuit, aby ST AN2867 Application Note, the value can be find by R_EXT = 1/ (2*pi*freq*C_load_Out) R_EXT = 530 ohm, smaller standar value is chosen The idea of R_EXT is to form a low pas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"
- note removed: "3 POWER INPUT 1* Normal (Lipo ~3.3-5V input) 2* High V (4.5V-12V input/USB 5V)"
- note removed: "CHECK EXTERNAL RESISTOR VALUE"
- note removed: "C_LOAD = 2*(C_L - C_STARY) = 2*(12pF - (5-6pF)) = 12pF C_LOAD is single load cap value C_L is given by manufractuer C_STRAY is the capacitacne of the board (5-6 pF by research)"
- moved on the sheet: C1, C2, C3, C4, C5, D1, D2, F1, FB1, J1, J2, J9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

Commit message: Updated PCB Layout
Parts:
- added C26, C27, C28: 10u, Capacitor_SMD:C_0805_2012Metric, symbol Device:C_Small
- added D3: LED_RED, LED_SMD:LED_0603_1608Metric, symbol Device:LED
- added F2: 250mA, Fuse:Fuse_1206_3216Metric, symbol Device:Polyfuse
- added R14, R17: 10k, Resistor_SMD:R_0603_1608Metric, symbol Device:R_Small
- added R15, R18: 13k, Resistor_SMD:R_0603_1608Metric, symbol Device:R_Small
- added R16: 1k, Resistor_SMD:R_0603_1608Metric, symbol Device:R_Small
- added U7, U8: MT9700, Package_TO_SOT_SMD:SOT-23-5, symbol All-in-one_custom:MT9700
- C10: footprint Capacitor_SMD:C_0402_1005Metric -> Capacitor_SMD:C_0603_1608Metric
- C11: footprint Capacitor_SMD:C_0603_1608Metric -> Capacitor_SMD:C_0402_1005Metric
- D2: value LED_RED -> LED_BLUE; footprint LED_SMD:LED_0402_1005Metric -> LED_SMD:LED_0603_1608Metric
- J3: footprint (none) -> All-in-one-custom:SD_Card_custom
- J4: footprint (none) -> All-in-one-custom:USB_C_16PIN
- R7: value 1k5 -> 1k
- SW1: footprint All-in-one-custom:SMNR4020-2.2UH -> All-in-one-custom:K3-2336D-F1
- SW2, SW3: footprint (none) -> All-in-one-custom:GT-TC029
Connections:
- net +12V: now also Q1.3 (D); no longer F1.1
- net +3.3V: now also SW3.1, C27.2, C28.2, U7.1 (VOUT), U8.1 (VOUT); no longer C4.2, C5.2, C8.1, D2.2 (A), L1.2, R5.1, U2.1 (OUT)
- net +BATT: now also F2.1; no longer U2.3 (EN), U2.4 (IN)
- net BUCK_VFB: now also R3.2; no longer R3.1
- net BUCK_VIN: now also D1.1 (K), F1.1, Q1.2 (S); no longer C1.1, C2.1, FB1.2, U1.3 (VIN), U1.5 (EN)
- net GND: now also J4.S1 (SHIELD), R3.1, R4.1, R5.2, C26.1, C27.1, C28.1, R14.1, R15.1, R16.1, R17.1, R18.1, U7.2 (GND), U8.2 (GND); no longer R3.2, R4.2, SW3.2, U3.44 (BOOT0)
- net at F1.2: now also FB1.1; no longer Q1.3 (D)
- net at D2.1 (K): now also R4.2; no longer R4.1
- new net: R15.2, U7.3 (SET)
- new net: C26.2, C8.1, D2.2 (A), R14.2, U2.1 (OUT), U7.4 (EN), U7.5 (VIN)
- new net: C1.1, C2.1, FB1.2, U1.3 (VIN), U1.5 (EN)
- new net: C4.2, C5.2, D3.2 (A), L1.2, R17.2, U8.4 (EN), U8.5 (VIN)
- new net: F2.2, U2.3 (EN), U2.4 (IN)
- new net: D3.1 (K), R16.2
- new net: R18.2, U8.3 (SET)
- new net BOOT0: R5.1, SW3.2, U3.44 (BOOT0)
- no-connect marks 29 -> 28
Other:
- note added: "LED foward voltage ~3V"
- note removed: "Blue LED foward voltage ~3V"
- moved on the sheet: C1, C2, C3, C4, C5, C6, C7, D1, F1, FB1, J1, J2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
