File: PCB/All-in-one/All-in-one.kicad_pcb (KiCad board)
At the start: 4 copper layers, 54 x 52.5 mm, 62 parts, among them J1 HIGH VOLTAGE, J2 Micro_SD_Card_Det, J3 USB_C_Receptacle_USB2.0, J4 I2C_1, J5 GPIO, J6 SWD, J7 Conn_01x02, J8 Conn_01x02, J9 UART_2, Q1 AO3401A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

Commit message: Updated CubeIDE Code and Reviewed All-in-one X01 PCB - updated PCB labelling (UART_1 is mis-labelled as UART_2 on both .sch   and PCB) - Tried STM32 programming with simple PWM code
Parts:
- J9: value UART_2 -> UART_1
Changed lines of the file:
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@@
       (effects (font (size 1 1) (thickness 0.15)))
     )
-    (fp_text value "UART_2" (at 2.6 4.2 90) (layer "F.SilkS")
+    (fp_text value "UART_1" (at 2.6 4.2 90) (layer "F.SilkS")
       (effects (font (size 1 1) (thickness 0.15)))
     )
@@
     (effects (font (size 1 1) (thickness 0.15)) (justify mirror))
   )
-  (gr_text "ALL-IN-ONE\nVER X01\nMADE BY GORDON SO\n16-SEP-2022" (at 58.3 29) (layer "B.SilkS")
+  (gr_text "ALL-IN-ONE\nVER X01\nMADE BY GORDON SO\n16-SEP-2022" (at 116.1 27) (layer "B.SilkS")
     (effects (font (size 1 1) (thickness 0.15)) (justify mirror))
   )
